File: Avionics-RWboard.kicad_pcb (KiCad board)
At the start: 2 copper layers, 0 parts

Commit message: Start layout, still missing some footprints
Parts:
- added C1: 10nF, Capacitor_SMD:C_0603_1608Metric, F.Cu at (256.5, 95.1)
- added C10: 47u, Capacitor_SMD:C_1206_3216Metric_Pad1.33x1.80mm_HandSolder, F.Cu at (223.3, 57.8)
- added C11: 3n3, Capacitor_SMD:C_0603_1608Metric, F.Cu at (242.3, 59.0)
- added C12: 10nF, Capacitor_SMD:C_0603_1608Metric, F.Cu at (226.5, 86.2)
- added C13: 10nF, Capacitor_SMD:C_0603_1608Metric, F.Cu at (226.5, 88.7)
- added C14: 1u, Capacitor_SMD:C_0603_1608Metric, F.Cu at (228.3, 56.5)
- added C15: 0.1u, Capacitor_SMD:C_0402_1005Metric_Pad0.74x0.62mm_HandSolder, F.Cu at (258.8, 60.3)
- added C16: 22u, Capacitor_SMD:C_1210_3225Metric_Pad1.33x2.70mm_HandSolder, F.Cu at (249.3, 67.4)
- added C17: 47u, Capacitor_SMD:C_1206_3216Metric_Pad1.33x1.80mm_HandSolder, F.Cu at (223.3, 61.1)
- added C18: 47u, Capacitor_SMD:C_1206_3216Metric_Pad1.33x1.80mm_HandSolder, F.Cu at (223.3, 64.5)
- added C19: 47u, Capacitor_SMD:C_1206_3216Metric_Pad1.33x1.80mm_HandSolder, F.Cu at (223.3, 67.8)
- added C2: 10nF, Capacitor_SMD:C_0603_1608Metric, F.Cu at (256.5, 97.6)
- added C20: 47u, Capacitor_SMD:C_1206_3216Metric_Pad1.33x1.80mm_HandSolder, F.Cu at (223.3, 71.2)
- added C21: 47u, Capacitor_SMD:C_1206_3216Metric_Pad1.33x1.80mm_HandSolder, F.Cu at (223.3, 74.5)
- added C22: 1u, Capacitor_SMD:C_0603_1608Metric, F.Cu at (228.3, 59.0)
- added C23: 1u, Capacitor_SMD:C_0603_1608Metric, F.Cu at (228.3, 61.5)
- added C25: 22u, Capacitor_SMD:C_0603_1608Metric, F.Cu at (228.3, 64.0)
- added C26: 10u, Capacitor_SMD:C_1206_3216Metric_Pad1.33x1.80mm_HandSolder, F.Cu at (253.2, 90.2)
- added C27: 1u, Capacitor_SMD:C_0603_1608Metric, F.Cu at (258.3, 83.0)
- added C28: 100n, Capacitor_SMD:C_0402_1005Metric_Pad0.74x0.62mm_HandSolder, F.Cu at (261.9, 90.8)
- added C29: 10u, Capacitor_SMD:C_1206_3216Metric_Pad1.33x1.80mm_HandSolder, F.Cu at (243.3, 70.3)
- added C3: 47u, Capacitor_SMD:C_1206_3216Metric_Pad1.33x1.80mm_HandSolder, F.Cu at (253.2, 83.5)
- added C32: 47u, Capacitor_SMD:C_1206_3216Metric_Pad1.33x1.80mm_HandSolder, F.Cu at (223.3, 77.9)
- added C33: 10u, Capacitor_SMD:C_1206_3216Metric_Pad1.33x1.80mm_HandSolder, F.Cu at (223.3, 81.2)
- added C34: 1u, Capacitor_SMD:C_0603_1608Metric, F.Cu at (232.3, 54.0)
- added C35: 100n, Capacitor_SMD:C_0402_1005Metric_Pad0.74x0.62mm_HandSolder, F.Cu at (236.7, 71.2)
- added C4: 47u, Capacitor_SMD:C_1206_3216Metric_Pad1.33x1.80mm_HandSolder, F.Cu at (253.2, 86.8)
- added C5: 1u, Capacitor_SMD:C_0603_1608Metric, F.Cu at (242.3, 54.0)
- added C6: 10u, Capacitor_SMD:C_1206_3216Metric_Pad1.33x1.80mm_HandSolder, F.Cu at (243.3, 67.0)
- added C7: 10n, Capacitor_SMD:C_0603_1608Metric, F.Cu at (242.3, 56.5)
- added C8: 47nF, Capacitor_SMD:C_0603_1608Metric, F.Cu at (228.3, 54.0)
- added C9: 47u, Capacitor_SMD:C_1206_3216Metric_Pad1.33x1.80mm_HandSolder, F.Cu at (223.3, 54.4)
- added D1: GREEN, LED_SMD:LED_0603_1608Metric, F.Cu at (248.3, 70.8)
- added D2: GREEN LED, LED_SMD:LED_0603_1608Metric, F.Cu at (228.3, 71.5)
- added D3: RED LED, LED_SMD:LED_0603_1608Metric, F.Cu at (228.3, 74.1)
- added D4: GREEN LED, LED_SMD:LED_0603_1608Metric, F.Cu at (228.3, 76.7)
- added D5: 10V, Diode_SMD:Nexperia_DSN1608-2_1.6x0.8mm, F.Cu at (258.6, 69.7)
- added D6: RED LED, LED_SMD:LED_0603_1608Metric, F.Cu at (228.3, 79.2)
- added F1: 2000mA, Fuse:Fuse_0603_1608Metric, F.Cu at (242.3, 61.5)
- added H1: MountingHole_Pad, MountingHole:MountingHole_3.2mm_M3_Pad_Via, F.Cu at (103.3, 50.7)
- added H2: MountingHole_Pad, MountingHole:MountingHole_3.2mm_M3_Pad_Via, F.Cu at (177.0, 50.7)
- added H3: MountingHole_Pad, MountingHole:MountingHole_3.2mm_M3_Pad_Via, F.Cu at (99.5, 136.4)
- added H4: MountingHole_Pad, MountingHole:MountingHole_3.2mm_M3_Pad_Via, F.Cu at (179.6, 136.4)
- added J1: 282834-2, Argus-Connectors:TE_282834-2, F.Cu at (264.5, 85.8)
- added J2: 200528-0100, Argus-Connectors:Molex_200528-0100_1x10-1MP_P1.00mm_Horizontal, F.Cu at (259.6, 76.6)
- added Q1: NX3008NBKS, Package_TO_SOT_SMD:SOT-363_SC-70-6, F.Cu at (252.4, 95.8)
- added Q10: MBT2222ADW1T1, Package_TO_SOT_SMD:SOT-363_SC-70-6, F.Cu at (222.4, 90.8)
- added Q11: NX3008NBKS, Package_TO_SOT_SMD:SOT-363_SC-70-6, F.Cu at (222.4, 94.7)
- added Q12: MBT2222ADW1T1, Package_TO_SOT_SMD:SOT-363_SC-70-6, F.Cu at (222.4, 98.7)
- added Q2: MBT2222ADW1T1, Package_TO_SOT_SMD:SOT-363_SC-70-6, F.Cu at (252.4, 99.8)
- added Q3: NX3008NBKS, Package_TO_SOT_SMD:SOT-363_SC-70-6, F.Cu at (252.4, 103.7)
- added Q4: MBT2222ADW1T1, Package_TO_SOT_SMD:SOT-363_SC-70-6, F.Cu at (252.4, 107.6)
- added Q5: IRLML2803, Package_TO_SOT_SMD:SOT-23, F.Cu at (254.8, 61.7)
- added Q9: NX3008NBKS, Package_TO_SOT_SMD:SOT-363_SC-70-6, F.Cu at (222.4, 86.9)
- added R1: 680R, Resistor_SMD:R_0603_1608Metric, F.Cu at (256.5, 100.1)
- added R10: 10k, Resistor_SMD:R_0603_1608Metric, F.Cu at (264.5, 97.6)
- added R11: 10k, Resistor_SMD:R_0603_1608Metric, F.Cu at (264.5, 100.1)
- added R12: 200k, Resistor_SMD:R_0603_1608Metric, F.Cu at (264.5, 102.6)
- added R13: 0R, Resistor_SMD:R_0805_2012Metric_Pad1.20x1.40mm_HandSolder, F.Cu at (232.7, 71.7)
- added R14: 10k, Resistor_SMD:R_0603_1608Metric, F.Cu at (232.3, 56.5)
- added R15: 51k, Resistor_SMD:R_0603_1608Metric, F.Cu at (242.3, 64.0)
- added R16: 11k, Resistor_SMD:R_0603_1608Metric, F.Cu at (246.3, 54.0)
- added R17: 453R, Resistor_SMD:R_0603_1608Metric, F.Cu at (246.3, 56.5)
- added R2: 100k, Resistor_SMD:R_0603_1608Metric, F.Cu at (256.5, 102.6)
- added R20: 2.7k, Resistor_SMD:R_0603_1608Metric, F.Cu at (246.3, 59.0)
- added R21: 10k, Resistor_SMD:R_0603_1608Metric, F.Cu at (246.3, 61.5)
- added R22: 4k7, Resistor_SMD:R_0603_1608Metric, F.Cu at (246.3, 64.0)
- added R23: 10k, Resistor_SMD:R_0603_1608Metric, F.Cu at (250.3, 54.0)
- added R24: 0R, Resistor_SMD:R_0603_1608Metric, F.Cu at (250.3, 56.5)
- added R25: 0R, Resistor_SMD:R_0603_1608Metric, F.Cu at (250.3, 59.0)
- added R26: 10k, Resistor_SMD:R_0603_1608Metric, F.Cu at (232.3, 59.0)
- added R27: 1k, Resistor_SMD:R_0603_1608Metric, F.Cu at (232.3, 61.5)
- added R28: 4k7, Resistor_SMD:R_0603_1608Metric, F.Cu at (232.3, 64.0)
- added R29: 1k, Resistor_SMD:R_0603_1608Metric, F.Cu at (236.3, 54.0)
- added R3: 10k, Resistor_SMD:R_0603_1608Metric, F.Cu at (256.5, 105.1)
- added R30: 470, Resistor_SMD:R_0603_1608Metric, F.Cu at (236.3, 56.5)
- added R31: 0R, Resistor_SMD:R_0603_1608Metric, F.Cu at (258.3, 85.5)
- added R32: 0.05R, Resistor_SMD:R_0805_2012Metric_Pad1.20x1.40mm_HandSolder, F.Cu at (254.7, 70.0)
- added R33: 1K, Resistor_SMD:R_0603_1608Metric, F.Cu at (250.3, 61.5)
- added R34: 680R, Resistor_SMD:R_0603_1608Metric, F.Cu at (226.5, 91.2)
- added R35: 100k, Resistor_SMD:R_0603_1608Metric, F.Cu at (226.5, 93.7)
- added R36: 10k, Resistor_SMD:R_0603_1608Metric, F.Cu at (226.5, 96.2)
- added R37: 10k, Resistor_SMD:R_0603_1608Metric, F.Cu at (230.5, 86.2)
- added R38: 200k, Resistor_SMD:R_0603_1608Metric, F.Cu at (230.5, 88.7)
- added R39: 0R, Resistor_SMD:R_0603_1608Metric, F.Cu at (230.5, 91.2)
- added R4: 10k, Resistor_SMD:R_0603_1608Metric, F.Cu at (260.5, 95.1)
- added R40: 0R, Resistor_SMD:R_0603_1608Metric, F.Cu at (230.5, 93.7)
- added R41: 680R, Resistor_SMD:R_0603_1608Metric, F.Cu at (230.5, 96.2)
- added R42: 100k, Resistor_SMD:R_0603_1608Metric, F.Cu at (234.5, 86.2)
- added R43: 10k, Resistor_SMD:R_0603_1608Metric, F.Cu at (234.5, 88.7)
- added R44: 10k, Resistor_SMD:R_0603_1608Metric, F.Cu at (234.5, 91.2)
- added R45: 200k, Resistor_SMD:R_0603_1608Metric, F.Cu at (234.5, 93.7)
- added R46: 0R, Resistor_SMD:R_0603_1608Metric, F.Cu at (258.3, 88.1)
- added R47: 0R, Resistor_SMD:R_0603_1608Metric, F.Cu at (258.3, 90.6)
- added R48: 10k, Resistor_SMD:R_0603_1608Metric, F.Cu at (236.3, 59.0)
- added R49: 22R, Resistor_SMD:R_2512_6332Metric_Pad1.40x3.35mm_HandSolder, F.Cu at (230.8, 67.7)
- added R5: 200k, Resistor_SMD:R_0603_1608Metric, F.Cu at (260.5, 97.6)
- added R50: 0R, Resistor_SMD:R_0805_2012Metric_Pad1.20x1.40mm_HandSolder, F.Cu at (232.7, 74.6)
- added R6: 0R, Resistor_SMD:R_0603_1608Metric, F.Cu at (260.5, 100.1)
- added R7: 0R, Resistor_SMD:R_0603_1608Metric, F.Cu at (260.5, 102.6)
- added R8: 680R, Resistor_SMD:R_0603_1608Metric, F.Cu at (260.5, 105.1)
- added R9: 100k, Resistor_SMD:R_0603_1608Metric, F.Cu at (264.5, 95.1)
- added REF**: Gauge_10mm_Type1_SilkScreenTop, Calibration_Scale:Gauge_10mm_Type1_SilkScreenTop, F.Cu at (35.1, 88.0)
- added REF**: Val**, mainboard:XYZ_cubesat-top, B.Cu at (50.3, 35.2)
- added REF**: Val**, mainboard:XYZ_cubesat-bot, B.Cu at (64.7, 34.1)
- added U2: TPS259621DDA, Package_SO:Texas_R-PDSO-G8_EP2.95x4.9mm_Mask2.4x3.1mm_ThermalVias, F.Cu at (256.6, 56.1)
- added U4: ADM1176-1ARMZ-R7, Package_SO:MSOP-10_3x3mm_P0.5mm, F.Cu at (256.0, 66.3)
- added kibuzzard-67C0A908: G***, kibuzzard-67C0A908, F.Cu at (52.3, 67.4)
Other:
- board outline added: 90.2 x 95.9 mm
- board text added: "ARGUS Cubesat Carnegie Mellon University Mainboard v3.0"
- board text added: "mainboard.v3.0"
