File: Power.kicad_sch (KiCad schematic)
At the start: 41 parts, among them Q5 IRLML2803, Q6 SiRA99DP, U2 TPS259621DDA, U4 ADM1176-1ARMZ-R7

Commit message: Local Stash
Changed lines of the file:
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@@
 (kicad_sch
-	(version 20231120)
+	(version 20250114)
 	(generator "eeschema")
-	(generator_version "8.0")
+	(generator_version "9.0")
 	(paper "A4")
 	(title_block
@@
 		(rev "1.0")
 	)
+	(text "Not sure of how to configure this"
+		(exclude_from_sim no)
+		(at 106.934 141.478 0)
+		(effects
+			(font
+				(size 1.27 1.27)
+				(color 255 0 0 1)
+			)
+		)
+	)
+	(text "I2C1 ADDR"
+		(exclude_from_sim no)
+		(at 107.188 136.398 0)
+		(effects
+			(font
+				(size 2.159 2.159)
+			)
+			(justify right bottom)
+		)
+	)
+	(text "0x??\n"
+		(exclude_from_sim no)
+		(at 97.536 139.954 0)
+		(effects
+			(font
+				(size 2.159 2.159)
+			)
+			(justify right bottom)
+		)
+	)
+	(text "Motor Enable"
+		(exclude_from_sim no)
+		(at 25.4 24.13 0)
+		(effects
+			(font
+				(size 2.54 2.54)
+				(thickness 0.508)
+				(bold yes)
+			)
+			(justify left bottom)
+		)
+	)
+	(text "F1 shall be replaced with a 0-Ohm jumper on flight builds."
+		(exclude_from_sim no)
+		(at 35.306 83.058 0)
+		(effects
+			(font
+				(size 1.27 1.27)
+				(color 255 0 0 1)
+			)
+			(justify left bottom)
+		)
+	)
+	(text "I_limit = V_limit / R_sense = 0.1V / 0.01 R = 10 A\nPower: I x I x R = 10 x 10 x 0.01 = 1 Watts worst case\n"
+		(exclude_from_sim no)
+		(at 87.884 126.238 0)
+		(effects
+			(font
+				(size 0.889 0.889)
+			)
+			(justify left top)
+		)
+	)
+	(text "Motor Power Monitor"
+		(exclude_from_sim no)
+		(at 25.908 101.092 0)
+		(effects
+			(font
+				(size 2.54 2.54)
+				(thickness 0.508)
+				(bold yes)
+			)
+			(justify left bottom)
+		)
+	)
+	(text "TPS259621 = Autoretry after thermal shutdown\nCard current limited to 2.0 A by R_ILM = 453 ohm\ndv/dt = 10nF sets it to 4.2 V/ms instead of the default 70 V/ms\nOVLO = 13.7 V (open)\nUVLO : Vin(UV) = Vuvlo(F) x (R1+R2)/(R2) = 1.1V x (51+11)/(11) = 6.2 V"
+		(exclude_from_sim no)
+		(at 203.2 72.898 0)
+		(effects
+			(font
+				(size 0.889 0.889)
+			)
+			(justify left)
+		)
+	)
+	(text "Fuse Bypass Jumpers"
+		(exclude_from_sim no)
+		(at 25.4 162.052 0)
+		(effects
+			(font
+				(size 2.54 2.54)
+				(thickness 0.508)
+				(bold yes)
+			)
+			(justify left bottom)
+		)
+	)
+	(text "Should be 0x46\n"
+		(exclude_from_sim no)
+		(at 98.298 143.51 0)
+		(effects
+			(font
+				(size 1.27 1.27)
+				(color 255 0 0 1)
+			)
+		)
+	)
+	(text "PI Filter"
+		(exclude_from_sim no)
+		(at 186.182 101.092 0)
+		(effects
+			(font
+				(size 2.54 2.54)
+				(thickness 0.508)
+				(bold yes)
+			)
+			(justify left bottom)
+		)
+	)
+	(text "Bypasses for the fuses\n"
+		(exclude_from_sim no)
+		(at 28.702 185.42 0)
+		(effects
+			(font
+				(size 1.27 1.27)
+				(color 0 0 194 1)
+			)
+			(justify left bottom)
+		)
+	)
+	(text "Motor eFuse\n"
+		(exclude_from_sim no)
+		(at 165.1 24.892 0)
+		(effects
+			(font
+				(size 2.54 2.54)
+				(thickness 0.508)
+				(bold yes)
+			)
+			(justify left bottom)
+		)
+	)
 	(junction
 		(at 147.32 109.22)
@@
 		)
 	)
-	(text "Not sure of how to configure this"
-		(exclude_from_sim no)
-		(at 106.934 141.478 0)
-		(effects
-			(font
-				(size 1.27 1.27)
-				(color 255 0 0 1)
-			)
-		)
-	)
-	(text "I2C1 ADDR"
-		(exclude_from_sim no)
-		(at 107.188 136.398 0)
-		(effects
-			(font
-				(size 2.159 2.159)
-			)
-			(justify right bottom)
-		)
-	)
-	(text "0x??\n"
-		(exclude_from_sim no)
-		(at 97.536 139.954 0)
-		(effects
-			(font
-				(size 2.159 2.159)
-			)
-			(justify right bottom)
-		)
-	)
-	(text "Motor Enable"
-		(exclude_from_sim no)
-		(at 25.4 24.13 0)
-		(effects
-			(font
-				(size 2.54 2.54)
-				(thickness 0.508)
-				(bold yes)
-			)
-			(justify left bottom)
-		)
-	)
-	(text "F1 shall be replaced with a 0-Ohm jumper on flight builds."
-		(exclude_from_sim no)
-		(at 35.306 83.058 0)
-		(effects
-			(font
-				(size 1.27 1.27)
-				(color 255 0 0 1)
-			)
-			(justify left bottom)
-		)
-	)
-	(text "I_limit = V_limit / R_sense = 0.1V / 0.01 R = 10 A\nPower: I x I x R = 10 x 10 x 0.01 = 1 Watts worst case\n"
-		(exclude_from_sim no)
-		(at 87.884 126.238 0)
-		(effects
-			(font
-				(size 0.889 0.889)
-			)
-			(justify left top)
-		)
-	)
-	(text "Motor Power Monitor"
-		(exclude_from_sim no)
-		(at 25.908 101.092 0)
-		(effects
-			(font
-				(size 2.54 2.54)
-				(thickness 0.508)
-				(bold yes)
-			)
-			(justify left bottom)
-		)
-	)
-	(text "TPS259621 = Autoretry after thermal shutdown\nCard current limited to 2.0 A by R_ILM = 453 ohm\ndv/dt = 10nF sets it to 4.2 V/ms instead of the default 70 V/ms\nOVLO = 13.7 V (open)\nUVLO : Vin(UV) = Vuvlo(F) x (R1+R2)/(R2) = 1.1V x (51+11)/(11) = 6.2 V"
-		(exclude_from_sim no)
-		(at 203.2 72.898 0)
-		(effects
-			(font
-				(size 0.889 0.889)
-			)
-			(justify left)
-		)
-	)
-	(text "Fuse Bypass Jumpers"
-		(exclude_from_sim no)
-		(at 25.4 162.052 0)
-		(effects
-			(font
-				(size 2.54 2.54)
-				(thickness 0.508)
-				(bold yes)
-			)
-			(justify left bottom)
-		)
-	)
-	(text "Should be 0x46\n"
-		(exclude_from_sim no)
-		(at 98.298 143.51 0)
-		(effects
-			(font
-				(size 1.27 1.27)
-				(color 255 0 0 1)
-			)
-		)
-	)
-	(text "PI Filter"
-		(exclude_from_sim no)
-		(at 186.182 101.092 0)
-		(effects
-			(font
-				(size 2.54 2.54)
-				(thickness 0.508)
-				(bold yes)
-			)
-			(justify left bottom)
-		)
-	)
-	(text "Bypasses for the fuses\n"
-		(exclude_from_sim no)
-		(at 28.702 185.42 0)
-		(effects
-			(font
-				(size 1.27 1.27)
-				(color 0 0 194 1)
-			)
-			(justify left bottom)
-		)
-	)
-	(text "Motor eFuse\n"
-		(exclude_from_sim no)
-		(at 165.1 24.892 0)
-		(effects
-			(font
-				(size 2.54 2.54)
-				(thickness 0.508)
-				(bold yes)
-			)
-			(justify left bottom)
-		)
-	)
 	(label "SWITCHED_POWER"
 		(at 130.81 35.56 0)
@@
 		(at 35.56 111.76)
 		(size 27.94 7.62)
+		(exclude_from_sim no)
+		(in_bom yes)
+		(on_board yes)
+		(dnp no)
 		(fields_autoplaced yes)
 		(stroke
